File: FlightComputer_CPU_V1.kicad_pcb (KiCad board)
At the start: 4 copper layers, 31.8 x 31.8 mm, 64 parts, among them J1 Conn_02x08_Odd_Even, J2 Conn_02x08_Odd_Even, U1 STM32H503CBUx, U2 LD2981-3.3, U3 MX25R6435FZNIL0, Y2 Crystal_GND24_Small

Commit message: Started Version 2
Parts:
- removed TP1, TP10, TP11, TP12, TP13, TP14, TP15, TP16, TP17, TP18, TP19, TP2, TP20, TP21, TP22, TP23, TP24, TP25, TP26, TP27, TP28, TP29, TP3, TP30, TP31, TP32, TP33, TP34, TP35, TP36, TP37, TP38, TP39, TP4, TP40, TP6, TP7, TP8, TP9: TestPoint, TestPoint:TestPoint_Pad_D1.0mm
- added J3: Male Front Left, Connector_PinHeader_1.27mm:PinHeader_2x08_P1.27mm_Vertical_SMD, F.Cu at (97.0, 69.8)
- added J4: Female Front Right, Connector_PinSocket_1.27mm:PinSocket_2x08_P1.27mm_Vertical_SMD, F.Cu at (119.0, 69.8)
- added R11: 4.7k, Resistor_SMD:R_0402_1005Metric, F.Cu at (102.6, 69.1)
- added R12: 4.7k, Resistor_SMD:R_0402_1005Metric, F.Cu at (102.6, 70.1)
- added R13: 4.7k, Resistor_SMD:R_0402_1005Metric, F.Cu at (113.2, 68.6)
- added R14: 4.7k, Resistor_SMD:R_0402_1005Metric, F.Cu at (110.2, 64.7)
- added R15: 1.2k, Resistor_SMD:R_0402_1005Metric, F.Cu at (107.7, 74.8)
- J1: value Conn_02x08_Odd_Even -> Female Back Left; footprint Connector_PinHeader_1.27mm:PinHeader_2x08_P1.27mm_Vertical -> Connector_PinSocket_1.27mm:PinSocket_2x08_P1.27mm_Vertical_SMD; moved to B.Cu
- J2: value Conn_02x08_Odd_Even -> Male Back Right; footprint Connector_PinHeader_1.27mm:PinHeader_2x08_P1.27mm_Vertical -> Connector_PinHeader_1.27mm:PinHeader_2x08_P1.27mm_Vertical_SMD; moved to B.Cu
- U3: value MX25R6435FZNIL0 -> W25Q128JVP; footprint Package_SON:WSON-8-1EP_6x5mm_P1.27mm_EP3.4x4mm -> Package_SON:WSON-8-1EP_6x5mm_P1.27mm_EP3.4x4.3mm
- moved C12 11.9 mm to (104.4, 74.5), turned to 180 degrees
- moved C14 8.79 mm to (105.2, 64.7), turned to 90 degrees
- moved C13 6.87 mm to (112.0, 65.7), turned to 180 degrees
- moved J1 5.02 mm to (97.0, 69.8), turned to 180 degrees
- moved R42 4.69 mm to (103.7, 59.9), turned to 180 degrees
- moved J2 4.57 mm to (119.0, 69.8), turned to 180 degrees
- moved R41 4.16 mm to (103.7, 60.9), turned to 180 degrees
- moved R40 4.07 mm to (103.7, 61.9), turned to 180 degrees
- moved C30 3.99 mm to (118.4, 77.6), turned to 90 degrees
- moved C10 3.16 mm to (102.6, 72.6), turned to 180 degrees
- moved D4 1.80 mm to (99.8, 60.9), turned to 0 degrees
- moved U3 1.62 mm to (114.6, 78.8), turned to 180 degrees
- moved C20 1.35 mm to (99.5, 76.6), turned to 0 degrees
- moved C17 1.10 mm to (107.4, 79.8)
- moved C18 1.10 mm to (105.4, 79.8), turned to 180 degrees
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Connections:
- C17 pad 1: /RCC_OSC_OUT -> Net-(C17-Pad1)
- Y2 pad 3: /RCC_OSC_OUT -> Net-(C17-Pad1)
Routing:
- net /SPI3_SCK: track 24.3 -> 0.81 mm, vias 2 -> 1
- net /SPI3_MISO: track 23.7 -> 0.81 mm, vias 2 -> 1
- net /I2C2_SDA: track 23.4 -> 5.11 mm
- net /IRQ_2: track 23.0 -> 5.03 mm, vias 1 -> 2
- net /I2C1_SCL: track 23.2 -> 5.52 mm, vias 1 -> 2
- net /IRQ_1: track 21.5 -> 3.97 mm
- net /I2C1_SDA: track 22.8 -> 5.31 mm, vias 2 -> 1
- net /USART1_RX: track 21.3 -> 4.55 mm, vias 1 -> 2
- net /USART2_RX: track 20.7 -> 4.80 mm, vias 1 -> 2
- net /SWDCLK: track 15.7 -> 1.31 mm, vias 0 -> 1
- net /LEDR: track 14.3 -> 0.81 mm, vias 2 -> 1
- net /USART1_TX: track 18.0 -> 4.80 mm, vias 1 -> 2
- net /FLASH_CS: track 14.1 -> 2.27 mm, vias 2 -> 1
- net /FDCAN1_RX: track 17.2 -> 5.62 mm, vias 1 -> 2
- net /SWDIO: track 12.7 -> 1.06 mm, vias 0 -> 1
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- added copper zone on In2.Cu, net +3V3_CPU
- removed copper zone on In2.Cu, net +5V
Other:
- board text added: "BOTTOM FACE"
- board text added: "Julien UHRY 10-2026"
- board text added: "STM32H5"
- board text removed: "+5V"
- board text removed: "3V3"
- board text removed: "BOTTOM"
- board text removed: "GND"
- board text removed: "Julien UHRY Sept 2026"
- board text removed: "LPRX"
- board text removed: "LPTX"
- board text removed: "MODULEX SYSTEM"
- board text removed: "RST"
- board text removed: "SIO"
- board text removed: "SLK"
- board text removed: "STM32H503CBUx"
- board text removed: "SWD Debug"
- board text removed: "TOP"
