File: FlightComputer_CPU_V1.kicad_sch (KiCad schematic)
At the start: 64 parts, among them J1 Conn_02x08_Odd_Even, J2 Conn_02x08_Odd_Even, U1 STM32H503CBUx, U2 LD2981-3.3, U3 MX25R6435FZNIL0, Y2 Crystal_GND24_Small

Commit message: Started Version 2
Parts:
- removed U3: MX25R6435FZNIL0, Package_SON:WSON-8-1EP_6x5mm_P1.27mm_EP3.4x4mm, symbol Memory_Flash:MX25R3235FZNxx0
- added J3: Male Front Left, Connector_PinHeader_1.27mm:PinHeader_2x08_P1.27mm_Vertical_SMD, symbol Connector_Generic:Conn_02x08_Odd_Even
- added J4: Female Front Right, Connector_PinSocket_1.27mm:PinSocket_2x08_P1.27mm_Vertical_SMD, symbol Connector_Generic:Conn_02x08_Odd_Even
- added R11, R12, R13, R14: 4.7k, Resistor_SMD:R_0402_1005Metric, symbol Device:R_Small
- added R15: 1.2k, Resistor_SMD:R_0402_1005Metric, symbol Device:R_Small
- added U3: W25Q128JVP, Package_SON:WSON-8-1EP_6x5mm_P1.27mm_EP3.4x4.3mm, symbol Memory_Flash:W25Q128JVP
- C30: now fitted; now in the parts list
- J1: value Conn_02x08_Odd_Even -> Female Back Left; footprint Connector_PinHeader_1.27mm:PinHeader_2x08_P1.27mm_Vertical -> Connector_PinSocket_1.27mm:PinSocket_2x08_P1.27mm_Vertical_SMD; now fitted; now in the parts list
- J2: value Conn_02x08_Odd_Even -> Male Back Right; footprint Connector_PinHeader_1.27mm:PinHeader_2x08_P1.27mm_Vertical -> Connector_PinHeader_1.27mm:PinHeader_2x08_P1.27mm_Vertical_SMD; now fitted; now in the parts list
Connections:
- net +3.3V: now also J3.2 (Pin_2)
- net +3V3_CPU: now also R11.2, R12.1, R13.1, R14.1, U3.3 (~{WP}/IO_{2}), U3.7 (~{HOLD}/~{RESET}/IO_{3}), U3.8 (VCC)
- net +5V: now also J3.14 (Pin_14), J3.3 (Pin_3), J4.14 (Pin_14), J4.3 (Pin_3)
- net FDCAN1_RX: now also J3.4 (Pin_4)
- net FDCAN1_TX: now also J3.6 (Pin_6)
- net FLASH_CS: now also U3.1 (~{CS})
- net GND: now also J3.1 (Pin_1), J3.16 (Pin_16), J4.1 (Pin_1), J4.16 (Pin_16), U3.4 (GND), U3.9 (EP)
- net GPIO_1: now also J4.5 (Pin_5)
- net GPIO_2: now also J3.12 (Pin_12)
- net GPIO_3: now also J3.10 (Pin_10)
- net I2C1_SCL: now also J4.11 (Pin_11), R12.2
- net I2C1_SDA: now also J4.13 (Pin_13), R11.1
- net I2C2_SCL: now also J4.7 (Pin_7), R13.2
- net I2C2_SDA: now also J4.9 (Pin_9), R14.2
- net IRQ_1: now also J3.5 (Pin_5)
- net IRQ_2: now also J3.7 (Pin_7)
- net RCC_OSC_OUT: now also R15.2; no longer C17.1, Y2.3
- net Reserved1: now also J3.15 (Pin_15)
- net Reserved2: now also J3.13 (Pin_13)
- net Reserved3: now also J3.11 (Pin_11)
- net SPI1_MISO: now also J4.10 (Pin_10)
- net SPI1_MOSI: now also J4.12 (Pin_12)
- net SPI1_SCK: now also J4.15 (Pin_15)
- net SPI3_MISO: now also U3.2 (DO/IO_{1})
- net SPI3_MOSI: now also U3.5 (DI/IO_{0})
- net SPI3_SCK: now also U3.6 (CLK)
- net USART1_RX: now also J4.2 (Pin_2)
- net USART1_TX: now also J4.4 (Pin_4)
- net USART2_RX: now also J4.6 (Pin_6)
- net USART2_TX: now also J4.8 (Pin_8)
- net VBat: now also J3.8 (Pin_8), J3.9 (Pin_9)
- new net: C17.1, R15.1, Y2.3
- no-connect marks 8 -> 15
Other:
- note added: "SPI Flash 128Mb"
- note removed: "Decoupling"
- note removed: "SPI Flash"
- moved on the sheet: C10, C11, C12, C13, C14, C15, C16, C17, C18, C20, C21, D4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
Changed lines of the file:
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@@
 	(generator_version "10.0")
 	(paper "A4")
+	(title_block
+		(date "2026-10-23")
+	)
